Commit message: cleaning up files and changing urdf paths

File: construction/panda_arm.urdf (robot description, URDF)
Before this commit: robot panda, 8 links, 7 joints
Links:
- added link linkTool, mass 1; visual mesh filename=../../../model/Drill2/Drill2.obj
- link link0: geometry visual mesh filename=../../../model/panda/meshes/visual/link0.obj
- link link1: geometry visual mesh filename=../../../model/panda/meshes/visual/link1.obj
- link link2: geometry visual mesh filename=../../../model/panda/meshes/visual/link2.obj
- link link3: geometry visual mesh filename=../../../model/panda/meshes/visual/link3.obj
- link link4: geometry visual mesh filename=../../../model/panda/meshes/visual/link4.obj
- link link5: geometry visual mesh filename=../../../model/panda/meshes/visual/link5.obj
- link link6: geometry visual mesh filename=../../../model/panda/meshes/visual/link6.obj
- link link7: geometry visual mesh filename=../../../model/panda/meshes/visual/link7.obj

Commit message: added drill files and added visuals to joint7

File: construction/panda_arm.urdf (robot description, URDF)
Before this commit: robot panda, 9 links, 7 joints
Links:
- removed link linkTool
- link link7: geometry visual mesh filename=../../../model/Drill2/Drill2.obj; visual mesh filename=../../../model/panda/meshes/visual/link7.obj
