Commit message: drill and wrench end effectors on panda arms. Have to fix mtl rendering

File: construction/panda_arm_wrench.urdf (robot description, URDF)
Before this commit: robot panda, 8 links, 7 joints
Links:
- link link7: geometry visual mesh filename=../../../model/Wrench/Wrench.obj; visual mesh filename=../../../model/panda/meshes/visual/link7.obj

Commit message: fixed glew rendering issue. Need to fix tool scaling

File: construction/panda_arm_wrench.urdf (robot description, URDF)
Before this commit: robot panda, 8 links, 7 joints
Links:
- link link7: geometry visual mesh filename=../../../model/Monkey_Wrench_v3/10299_Monkey-Wrench_v1_L3.o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; visual mesh filename=../../../model/panda/meshes/visual/link7.obj

Commit message: collision active for column object

File: construction/panda_arm_wrench.urdf (robot description, URDF)
Before this commit: robot panda, 8 links, 7 joints
Links:
- link link7: geometry collision mesh filename=../../../model/Monkey_Wrench_v3/10299_Monkey-Wrench_v1_L3.o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 scale=0.011 0.011 0.011; visual mesh filename=../../../model/Monkey_Wrench_v3/10299_Monkey-Wrench_v1_L3.o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 scale=0.011 0.011 0.011
