Commit message: cool tools working

File: construction/panda_arm_drill.urdf (robot description, URDF)
Before this commit: robot panda, 8 links, 7 joints
Links:
- link link7: geometry collision mesh filename=../../../model/cordless_drill/10108_Cordless Drill_v2_Itera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 scale=0.011 0.011 0.011; visual mesh filename=../../../model/cordless_drill/10108_Cordless Drill_v2_Itera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 scale=0.011 0.011 0.011

File: construction/panda_arm_wrench.urdf (robot description, URDF)
Before this commit: robot panda, 8 links, 7 joints
Links:
- link link7: geometry visual mesh filename=../../../model/Monkey_Wrench_v3/10299_Monkey-Wrench_v1_L3.o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 scale=0.011 0.011 0.011; visual mesh filename=../../../model/panda/meshes/visual/link7.obj

Commit message: modified drill to hilti

File: construction/panda_arm_drill.urdf (robot description, URDF)
Before this commit: robot panda, 8 links, 7 joints
Links:
- link link7: geometry collision mesh filename=../../../model/Hiltidrill/hiltidrill.obj scale=1 1 1; visual mesh filename=../../../model/Hiltidrill/hiltidrill.obj scale=1 1 1
