Commit message: weld tool

File: weld/mmp_panda3.urdf (robot description, URDF)
Before this commit: robot mmp_panda, 14 links, 13 joints
Links:
- link linkTool: geometry visual mesh filename=../../../model/weldtool/weldtool.obj

Commit message: improved joint example

File: weld/mmp_panda3.urdf (robot description, URDF)
Before this commit: robot mmp_panda, 14 links, 13 joints
Links:
- link base_z: geometry visual mesh filename=../../../model/mmp_panda_tall/meshes/panda_base.obj

Commit message: working demo for welding

File: weld/mmp_panda3.urdf (robot description, URDF)
Before this commit: robot mmp_panda, 14 links, 13 joints
Links:
- removed link base_fix
- removed link base_z
- added link base_link, mass 64.6; visual mesh filename=../../../model/mmp_panda_tall/meshes/panda_base.obj
- link linkTool: geometry collision cylinder length=0.24 radius=0.015; visual mesh filename=../../../model/weldtool/weldtool.obj
Joints:
- removed joint base_prismatic_z
- joint base_fixed: child base_fix -> base_link; origin xyz=0 0 0 rpy=0 0 1.57079632679 -> xyz=0 0 0.15 rpy=0 0 1.57079632679
- joint base_prismatic_x: origin xyz=0 0 0 rpy=0 0 0 -> xyz=-2.5 -0.2 0 rpy=0 0 0
- joint joint1: origin xyz=0 0 0.333 rpy=0 0 1.5708 -> xyz=0 0 0.333 rpy=0 0 0; parent base_z -> base_link
