Commit message: new panda

File: joint/mmp_panda2.urdf (robot description, URDF)
Before this commit: robot mmp_panda, 6 links, 5 joints
Links:
- link base_theta: geometry visual mesh filename=../../../model/jointcart2/joint cart2.obj
- link base_z: geometry visual mesh filename=../../../model/jointcart2/joint cart2.obj

Commit message: Added flaps and cut the speed

File: joint/mmp_panda2.urdf (robot description, URDF)
Before this commit: robot mmp_panda, 6 links, 5 joints
Links:
- link linkTool: geometry collision box size=0.16 0.02 0.01; collision cylinder length=0.1 radius=0.01

Commit message: Changed link tool joint orientation

File: joint/mmp_panda2.urdf (robot description, URDF)
Before this commit: robot mmp_panda, 6 links, 5 joints
Links:
- link linkTool: geometry collision box size=0.16 0.02 0.01; collision cylinder length=0.1 radius=0.01
Joints:
- joint jointTool: origin xyz=0 0 0 rpy=0 0 2 -> xyz=0 0 0 rpy=0 0 1.57

Commit message: Fixed flap so sensor doesn't impede motion

File: joint/mmp_panda2.urdf (robot description, URDF)
Before this commit: robot mmp_panda, 6 links, 5 joints
Links:
- link linkTool: geometry collision box size=0.08 0.02 0.01; collision cylinder length=0.1 radius=0.01

Commit message: Changed robot base

File: joint/mmp_panda2.urdf (robot description, URDF)
Before this commit: robot mmp_panda, 6 links, 5 joints
Links:
- link base_theta: geometry visual mesh filename=../../../model/jointcart2/jointcart2_wheeled.obj
Joints:
- joint base_fixed: origin xyz=0 0 0 rpy=0 0 1.57079632679 -> xyz=0 0 0.01 rpy=0 0 1.57079632679
- joint base_prismatic_x: origin xyz=0 0 0 rpy=0 0 0 -> xyz=0 0 0.01 rpy=0 0 0
- joint base_prismatic_y: origin xyz=0 0 0 rpy=0 0 0 -> xyz=0 0 0.01 rpy=0 0 0
- joint base_revolute: origin xyz=0 0 0.0 rpy=0 0 0 -> xyz=0 0 0.01 rpy=0 0 0
- joint jointTool: origin xyz=0 0 0 rpy=0 0 1.57 -> xyz=0 0 0.01 rpy=0 0 1.57
