Commit message: Added fetch as robot base to both joint_autonomous and joint_haptics. Materials could be better

File: joint_autonomous/joint_robot.urdf (robot description, URDF)
Before this commit: robot mmp_panda, 6 links, 5 joints
Links:
- link base_theta: geometry visual mesh filename=../../../model/jointcart_fetch/jointcart_fetch.obj
